File: AG_TOOL#1.kicad_pcb (KiCad board)
At the start: 2 copper layers, 120 x 74.4 mm, 32 parts, among them J1 CONN_01X02, P1 CONN_01X03, P2 CONN_01X02, Q1 Q_NPN_Darlington_BCE, Q2 Q_PMOS_DGS, SW1 SW_Push, SW2 SW_Push, SW3 SW_Push, SW4 SW_Push, SW5 SW_Push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

Commit message: Adding in another fuse for the 120v line and a choke for the dc output
Parts:
- added F2: Fuse, Fuse_Holders_and_Fuses:Fuseholder_ATO_Blade_littlefuse_Pudenz_2_Pin, F.Cu at (197.7, 62.2)
- added L1: 2100HT-121-V-RC, Choke_Toroid_ThroughHole:Choke_Toroid_horizontal_Diameter3-5mm_Amidon-T12, F.Cu at (135.9, 75.5)
- moved T1 7.20 mm to (174.8, 70.9)
Connections:
- D1 pad 1: +12V -> Net-(D1-Pad1)
- T1 pad 2: 120V_L -> Net-(F2-Pad1)
Changed lines of the file:
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@@
 (kicad_pcb (version 4) (host pcbnew 4.0.6+dfsg1-1)
   (general
-    (links 75)
-    (no_connects 75)
+    (links 77)
+    (no_connects 77)
     (area 99.924999 24.924999 220.075001 99.475001)
     (thickness 1.6)
@@
     (tracks 0)
     (zones 0)
-    (modules 32)
-    (nets 69)
+    (modules 34)
+    (nets 71)
   )
   (page A4)
@@
   (net 67 "Net-(U3-Pad37)")
   (net 68 "Net-(U3-Pad38)")
+  (net 69 "Net-(D1-Pad1)")
+  (net 70 "Net-(F2-Pad1)")
   (net_class Default "This is the default net class."
     (clearance 0.2)
@@
     (add_net LCD_D7)
     (add_net MENU)
+    (add_net "Net-(D1-Pad1)")
     (add_net "Net-(D1-Pad3)")
     (add_net "Net-(D1-Pad4)")
@@
     (add_net "Net-(DS1-Pad9)")
     (add_net "Net-(F1-Pad2)")
+    (add_net "Net-(F2-Pad1)")
     (add_net "Net-(Q1-Pad1)")
     (add_net "Net-(Q1-Pad2)")
@@
     (fp_line (start -2.6 13.4) (end -2.6 -2.6) (layer F.SilkS) (width 0.15))
     (pad 1 thru_hole circle (at 0 0 90) (size 2.1 2.1) (drill 1.2) (layers *.Cu *.Mask)
-      (net 2 +12V))
+      (net 69 "Net-(D1-Pad1)"))
     (pad 2 thru_hole circle (at 0 10.8 90) (size 2.1 2.1) (drill 1.2) (layers *.Cu *.Mask)
       (net 1 GND))
@@
   )
   (module F10-110-C2:F10-110-C2 (layer F.Cu)
-    (at 182 71 90)
+    (at 174.8 70.9 90)
     (fp_text reference T1 (at 0 21.5 90) (layer F.SilkS)
       (effects (font (size 1 1) (thickness 0.15)))
@@
       (net 19 120V_N))
     (pad 2 thru_hole circle (at 10.0965 15.24 90) (size 2.54 2.54) (drill 1.524) (layers *.Cu *.Mask)
-      (net 20 120V_L))
+      (net 70 "Net-(F2-Pad1)"))
     (pad 6 thru_hole circle (at 10.0965 -15.24 90) (size 2.54 2.54) (drill 1.524) (layers *.Cu *.Mask)
       (net 17 "Net-(F1-Pad2)"))
@@
       (net 44 TC1-))
   )
+  (module Fuse_Holders_and_Fuses:Fuseholder_ATO_Blade_littlefuse_Pudenz_2_Pin (layer F.Cu)
+    (at 197.7 62.2 270)
+    (descr "Fuseholder ATO Blade littlefuse Pudenz 2 Pin")
+    (tags "Fuseholder ATO Blade littlefuse Pudenz 2 Pin")
+    (fp_text reference F2 (at 4.57 -2.78 270) (layer F.SilkS)
+      (effects (font (size 1 1) (thickness 0.15)))
+    )
+    (fp_text value Fuse (at 5.07 5.22 270) (layer F.Fab)
+      (effects (font (size 1 1) (thickness 0.15)))
+    )
+    (fp_line (start -5.35 -1.75) (end 14.55 -1.75) (layer F.Fab) (width 0.1))
+    (fp_line (start 14.55 -1.75) (end 14.55 4.15) (layer F.Fab) (width 0.1))
+    (fp_line (start 14.55 4.15) (end -5.35 4.15) (layer F.Fab) (width 0.1))
+    (fp_line (start -5.35 4.15) (end -5.35 -1.75) (layer F.Fab) (width 0.1))
+    (fp_line (start -5.4 -1.8) (end -0.81 -1.8) (layer F.SilkS) (width 0.12))
+    (fp_line (start 14.6 -1.8) (end 14.6 4.2) (layer F.SilkS) (width 0.12))
+    (fp_line (start 14.6 4.2) (end -5.4 4.2) (layer F.SilkS) (width 0.12))
+    (fp_line (start -5.4 4.2) (end -5.4 -1.8) (layer F.SilkS) (width 0.12))
+    (fp_line (start 0.81 -1.8) (end 8.38 -1.8) (layer F.SilkS) (width 0.12))
+    (fp_line (start -5.65 -2.05) (end 14.85 -2.05) (layer F.CrtYd) (width 0.05))
+    (fp_line (start -5.65 -2.05) (end -5.65 4.45) (layer F.CrtYd) (width 0.05))
+    (fp_line (start 14.85 4.45) (end 14.85 -2.05) (layer F.CrtYd) (width 0.05))
+    (fp_line (start 14.85 4.45) (end -5.65 4.45) (layer F.CrtYd) (width 0.05))
+    (fp_line (start 10.02 -1.8) (end 14.6 -1.8) (layer F.SilkS) (width 0.12))
+    (pad 1 thru_hole circle (at 0 0 270) (size 3.5 3.5) (drill 2) (layers *.Cu *.Mask)
+      (net 70 "Net-(F2-Pad1)"))
+    (pad "" thru_hole circle (at 4.6 1.2 270) (size 2.4 2.4) (drill 2.4) (layers *.Cu *.Mask))
+    (pad 2 thru_hole circle (at 9.2 0 270) (size 3.5 3.5) (drill 2) (layers *.Cu *.Mask)
+      (net 20 120V_L))
+  )
+  (module Choke_Toroid_ThroughHole:Choke_Toroid_horizontal_Diameter3-5mm_Amidon-T12 (layer F.Cu)
+    (at 135.9 75.5 180)
+    (descr "Choke, Inductance, Toroid, horizontal, laying, Diameter 3,5mm, Amidon, T12,")
+    (tags "Choke, Inductance, Toroid, horizontal, laying, Diameter 3,5mm, Amidon, T120,")
+    (fp_text reference L1 (at 0 -3.81 180) (layer F.SilkS)
+      (effects (font (size 1 1) (thickness 0.15)))
+    )
+    (fp_text value 2100HT-121-V-RC (at 0 3.81 180) (layer F.Fab)
+      (effects (font (size 1 1) (thickness 0.15)))
+    )
+    (fp_line (start -1.80086 0) (end -0.8001 0) (layer F.SilkS) (width 0.15))
+    (fp_line (start -0.8001 0) (end -1.50114 0.8001) (layer F.SilkS) (width 0.15))
+    (fp_line (start -1.50114 0.8001) (end -0.59944 0.50038) (layer F.SilkS) (width 0.15))
+    (fp_line (start -0.59944 0.50038) (end -0.8001 1.50114) (layer F.SilkS) (width 0.15))
+    (fp_line (start -0.8001 1.50114) (end -0.09906 0.70104) (layer F.SilkS) (width 0.15))
+    (fp_line (start -0.09906 0.70104) (end -0.09906 1.69926) (layer F.SilkS) (width 0.15))
+    (fp_line (start -0.09906 1.69926) (end 0.29972 0.59944) (layer F.SilkS) (width 0.15))
+    (fp_line (start 0.29972 0.59944) (end 1.00076 1.39954) (layer F.SilkS) (width 0.15))
+    (fp_line (start 1.00076 1.39954) (end 0.59944 0.39878) (layer F.SilkS) (width 0.15))
+    (fp_line (start 0.59944 0.39878) (end 1.50114 0.70104) (layer F.SilkS) (width 0.15))
+    (fp_line (start 1.50114 0.70104) (end 0.8001 0) (layer F.SilkS) (width 0.15))
+    (fp_line (start 0.8001 0) (end 1.69926 0) (layer F.SilkS) (width 0.15))
+    (fp_circle (center 0 0) (end 0.70104 0) (layer F.SilkS) (width 0.15))
+    (fp_circle (center 0 0) (end 1.80086 0) (layer F.SilkS) (width 0.15))
+    (fp_text user End (at 8.19912 -2.90068 180) (layer F.SilkS)
+      (effects (font (size 1 1) (thickness 0.15)))
+    )
+    (fp_text user Start (at -8.60044 -2.90068 180) (layer F.SilkS)
+      (effects (font (size 1 1) (thickness 0.15)))
+    )
+    (pad 1 thru_hole circle (at -3.29946 0 180) (size 1.99898 1.99898) (drill 0.8001) (layers *.Cu *.Mask)
+      (net 69 "Net-(D1-Pad1)"))
+    (pad 2 thru_hole circle (at 3.29946 0 180) (size 1.99898 1.99898) (drill 0.8001) (layers *.Cu *.Mask)
+      (net 2 +12V))
+  )
   (gr_line (start 100 99.4) (end 220 99.4) (angle 90) (layer Edge.Cuts) (width 0.15))

Commit message: well i need to go to sleep now but i added in a din connector for the heater output and started routing a little it's comming together nicely
Parts:
- J1: value CONN_01X02 -> CONN_01X03; footprint k_ansi_thermocouple_Socket_pcb:K_ANSI_THERMOCOUPLE_SOCKET_PCB -> SDF-30J:SDF-30J
- RL1: footprint Capacitors_THT:CP_Radial_D22.0mm_P10.00mm_3pin_SnapIn -> SIP_SSR_CRYDOM:MCX240A5R
- moved RL1 83.1 mm to (138.4, 82.9), turned to 0 degrees
- moved P2 54.7 mm to (112.7, 33.5)
- moved J1 46.1 mm to (109.1, 80.8), turned to 270 degrees
- moved Q2 26.5 mm to (170.0, 51.0), turned to 90 degrees
- moved R6 16.9 mm to (170.0, 46.0)
- moved Q1 16.4 mm to (174.7, 47.4), turned to 0 degrees
- moved R7 15.0 mm to (170.0, 48.0), turned to 0 degrees
- moved C2 11.7 mm to (110.3, 60.8)
- moved L1 10.5 mm to (125.5, 76.8)
- moved R3 10.1 mm to (144.0, 47.0)
- moved F1 6.41 mm to (153.0, 59.4)
- moved C1 5.87 mm to (129.8, 64.7)
- moved D1 4.70 mm to (139.3, 75.1)
- moved R1 3.69 mm to (114.0, 47.0)
- moved U1 2.50 mm to (115.8, 62.5), turned to 270 degrees
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Connections:
- J1 pad 1: TC1+ -> 120V_N
- J1 pad 2: TC1- -> Net-(J1-Pad2)
- P2 pad 1: TO_HTR -> TC1+
- P2 pad 2: 120V_N -> TC1-
Routing:
- net GND: track 0.00 -> 120.0 mm
- net 120V_N: track 0.00 -> 105.7 mm
- net +12V: track 0.00 -> 88.1 mm
- net 120V_L: track 0.00 -> 81.3 mm
- net +5V: track 0.00 -> 71.3 mm
- net TO_SSR: track 0.00 -> 51.2 mm, vias 0 -> 1
- net Net-(D1-Pad4): track 0.00 -> 28.2 mm
- net LCD_D6: track 0.00 -> 28.0 mm
- net Earth: track 0.00 -> 23.5 mm
- net TO_HTR: track 0.00 -> 19.3 mm
- net +3V3: track 0.00 -> 15.8 mm
- net LCD_D7: track 0.00 -> 11.7 mm
- net Net-(D1-Pad1): track 0.00 -> 11.2 mm
- net LCD_D5: track 0.00 -> 9.58 mm
- net Net-(F2-Pad1): track 0.00 -> 8.24 mm
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Other:
- net class 120V added: clearance 0.2, trace_width 2.75, via_dia 2.75, via_drill 2.5
- net class 12v added: clearance 0.2, trace_width 0.25, via_dia 0.6, via_drill 0.4

Commit message: changed some parts
Parts:
- DS1: footprint Pin_Headers:Pin_Header_Angled_2x16_Pitch2.00mm -> Pin_Headers:Pin_Header_Straight_1x16_Pitch2.00mm
- moved U3 38.1 mm to (173.0, 40.0), turned to 270 degrees
- moved Q1 22.6 mm to (195.7, 39.0)
- moved Q2 22.6 mm to (191.0, 42.6)
- moved R6 22.6 mm to (191.0, 37.6)
- moved R7 22.6 mm to (191.0, 39.6)
- moved DS1 22.5 mm to (157.4, 33.6)
Connections:
- U3 pad 27: Net-(U3-Pad27) -> TEMP-
- U3 pad 29: Net-(U3-Pad29) -> MENU
- U3 pad 3: Net-(U3-Pad3) -> TEMP+
- U3 pad 5: Net-(U3-Pad5) -> FORWARD
- U3 pad 7: Net-(U3-Pad7) -> BACK
Routing:
- net +5V: track 71.3 -> 12.4 mm
- net +12V: track 88.1 -> 34.9 mm
- net GND: track 120.0 -> 90.0 mm
- net LCD_D6: track 28.0 -> 0.00 mm
- net TO_SSR: track 51.2 -> 27.4 mm
- net +3V3: track 15.8 -> 0.00 mm
- net LCD_D7: track 11.7 -> 0.00 mm
- net LCD_D5: track 9.58 -> 0.00 mm
- net TO_MFET: track 6.60 -> 0.10 mm
- net LCD_D4: track 6.41 -> 0.00 mm
- net Net-(R1-Pad1): track 3.63 -> 0.00 mm
- net Net-(Q1-Pad2): track 7.87 -> 4.47 mm
- net Net-(R4-Pad1): track 3.13 -> 0.00 mm
- net Net-(R5-Pad1): track 3.13 -> 0.00 mm
- net Net-(R3-Pad1): track 3.13 -> 0.00 mm
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- added copper zone on B.Cu, net GND
Other:
- net class 12v: clearance 0.2 -> 0.155; trace_width 0.25 -> 0.155
- rule trace_min: 0.2 -> 0.155
- rule via_min_drill: 0.3 -> 0.4
- rule via_min_size: 0.4 -> 0.5
