File: AG_TOOL#1.sch (KiCad schematic (older format))
At the start: 33 parts, among them J1 CONN_01X02, P1 CONN_01X03, P2 CONN_01X02, Q1 Q_NPN_Darlington_BCE, Q2 Q_PMOS_DGS, SW1 SW_Push, SW2 SW_Push, SW3 SW_Push, SW4 SW_Push, SW5 SW_Push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

Commit message: Adding in another fuse for the 120v line and a choke for the dc output
Parts:
- added F2: Fuse, Fuse_Holders_and_Fuses:Fuseholder_ATO_Blade_littlefuse_Pudenz_2_Pin, symbol Fuse
- added L1: 2100HT-121-V-RC, Choke_Toroid_ThroughHole:Choke_Toroid_horizontal_Diameter3-5mm_Amidon-T12, symbol L_Core_Iron_Small
Connections:
- net +12V: now also L1.2; no longer D1.1 (+)
- net 120V_L: now also F2.2; no longer T1.2 (AB)
- new net: D1.1 (+), L1.1
- new net: F2.1, T1.2 (AB)
Changed lines of the file:
@@
 LIBS:pspice
 LIBS:switches
-LIBS:ERGO_V5-cache
 EELAYER 25 0
 EELAYER END
@@
 Text GLabel 2450 1350 0    60   Input ~ 0
 120V_N
-Text GLabel 3750 950  0    60   Input ~ 0
+Text GLabel 3450 950  0    60   Input ~ 0
 120V_L
 Text GLabel 3750 1350 0    60   Input ~ 0
@@
 P 5800 1150
 F 0 "D1" H 5850 1425 50  0000 L CNN
-F 1 "D_Bridge_+-AA" H 5850 1350 50  0000 L CNN
+F 1 "D_Bridge_+-AA" H 5600 1550 50  0000 L CNN
 F 2 "Diodes_THT:Diode_Bridge_15.7x15.7" H 5800 1150 50  0001 C CNN
 F 3 "" H 5800 1150 50  0000 C CNN
@@
 $EndComp
 $Comp
-L +12V #PWR28
+L +12V #PWR33
 U 1 1 593C44E1
-P 6100 1150
-F 0 "#PWR28" H 6100 1000 50  0001 C CNN
-F 1 "+12V" H 6100 1290 50  0000 C CNN
-F 2 "" H 6100 1150 50  0000 C CNN
-F 3 "" H 6100 1150 50  0000 C CNN
-	1    6100 1150
-	0    1    1    0
+P 6300 1150
+F 0 "#PWR33" H 6300 1000 50  0001 C CNN
+F 1 "+12V" H 6300 1300 50  0000 C CNN
+F 2 "" H 6300 1150 50  0000 C CNN
+F 3 "" H 6300 1150 50  0000 C CNN
+	1    6300 1150
+	-1   0    0    1
 $EndComp
 $Comp
@@
 $EndComp
 $Comp
-L GND #PWR33
+L GND #PWR32
 U 1 1 593C4CB9
 P 6250 5500
-F 0 "#PWR33" H 6250 5250 50  0001 C CNN
+F 0 "#PWR32" H 6250 5250 50  0001 C CNN
 F 1 "GND" H 6250 5350 50  0000 C CNN
 F 2 "" H 6250 5500 50  0000 C CNN
@@
 $EndComp
 $Comp
-L GND #PWR30
+L GND #PWR29
 U 1 1 593C4CDD
 P 6150 5500
-F 0 "#PWR30" H 6150 5250 50  0001 C CNN
+F 0 "#PWR29" H 6150 5250 50  0001 C CNN
 F 1 "GND" H 6150 5350 50  0000 C CNN
 F 2 "" H 6150 5500 50  0000 C CNN
@@
 DRDY
 $Comp
-L GND #PWR31
+L GND #PWR30
 U 1 1 593C766D
 P 6200 6900
-F 0 "#PWR31" H 6200 6650 50  0001 C CNN
+F 0 "#PWR30" H 6200 6650 50  0001 C CNN
 F 1 "GND" H 6200 6750 50  0000 C CNN
 F 2 "" H 6200 6900 50  0000 C CNN
@@
 BACK
 $Comp
-L +3.3V #PWR32
+L +3.3V #PWR31
 U 1 1 593C9516
 P 6250 2900
-F 0 "#PWR32" H 6250 2750 50  0001 C CNN
+F 0 "#PWR31" H 6250 2750 50  0001 C CNN
 F 1 "+3.3V" H 6250 3040 50  0000 C CNN
 F 2 "" H 6250 2900 50  0000 C CNN
@@
 $EndComp
 $Comp
-L +3.3V #PWR29
+L +3.3V #PWR28
 U 1 1 593C95AA
 P 6150 2900
-F 0 "#PWR29" H 6150 2750 50  0001 C CNN
+F 0 "#PWR28" H 6150 2750 50  0001 C CNN
 F 1 "+3.3V" H 6150 3040 50  0000 C CNN
 F 2 "" H 6150 2900 50  0000 C CNN
@@
 Text GLabel 3350 6550 0    60   Input ~ 0
 TC1+
+$Comp
+L L_Core_Iron_Small L1
+U 1 1 59985A6A
+P 6200 1150
+F 0 "L1" H 6250 1190 50  0000 L CNN
+F 1 "2100HT-121-V-RC" V 6400 750 50  0000 L CNN
+F 2 "Choke_Toroid_ThroughHole:Choke_Toroid_horizontal_Diameter3-5mm_Amidon-T12" H 6200 1150 50  0001 C CNN
+F 3 "" H 6200 1150 50  0001 C CNN
+	1    6200 1150
+	0    -1   -1   0
+$EndComp
+$Comp
+L Fuse F2
+U 1 1 59985D93
+P 3600 950
+F 0 "F2" V 3680 950 50  0000 C CNN
+F 1 "Fuse" V 3525 950 50  0000 C CNN
+F 2 "Fuse_Holders_and_Fuses:Fuseholder_ATO_Blade_littlefuse_Pudenz_2_Pin" V 3530 950 50  0001 C CNN
+F 3 "" H 3600 950 50  0001 C CNN
+	1    3600 950
+	0    1    1    0
+$EndComp
 $EndSCHEMATC

Commit message: well i need to go to sleep now but i added in a din connector for the heater output and started routing a little it's comming together nicely
Parts:
- removed J1: CONN_01X02, k_ansi_thermocouple_Socket_pcb:K_ANSI_THERMOCOUPLE_SOCKET_PCB, symbol CONN_01X02
- added J1: CONN_01X03, SDF-30J:SDF-30J, symbol CONN_01X03
Connections:
- net 120V_N: now also J1.1 (P1); no longer P2.2 (P2)
- net TC1+: now also P2.1 (P1)
- net TC1-: now also P2.2 (P2)
- net TO_HTR: now also J1.3 (P3); no longer P2.1 (P1)
Other:
- moved on the sheet: P2

Commit message: changed some parts
Parts:
- DS1: footprint Pin_Headers:Pin_Header_Angled_2x16_Pitch2.00mm -> Pin_Headers:Pin_Header_Straight_2x08_Pitch2.00mm
Connections:
- net BACK: now also U3.7 ((GCLK)_GPIO4)
- net FORWARD: now also U3.5 ((SCL1)_GPIO3)
- net MENU: now also U3.29 (GPIO5)
- net TEMP+: now also U3.3 ((SDA1)_GPIO2)
- net TEMP-: now also U3.27 (ID_SD)
Changed lines of the file:
@@
 LIBS:pspice
 LIBS:switches
+LIBS:AG_TOOL#1-cache
 EELAYER 25 0
 EELAYER END
@@
 F 0 "DS1" H 1900 4600 50  0000 C CNN
 F 1 "LCD16X2" H 3400 4600 50  0000 C CNN
-F 2 "Pin_Headers:Pin_Header_Angled_2x16_Pitch2.00mm" H 2700 4150 50  0001 C CIN
+F 2 "Pin_Headers:Pin_Header_Straight_2x08_Pitch2.00mm" H 2700 4150 50  0001 C CIN
 F 3 "" H 2700 4200 50  0000 C CNN
 	1    2700 4200
@@
 	1    0    0    -1
 $EndComp
+Text GLabel 6950 3300 2    60   Input ~ 0
+TEMP+
+Text GLabel 5150 4900 0    60   Input ~ 0
+TEMP-
+Text GLabel 6950 3700 2    60   Input ~ 0
+MENU
+Text GLabel 6950 3400 2    60   Input ~ 0
+FORWARD
+Text GLabel 6950 3500 2    60   Input ~ 0
+BACK
 $EndSCHEMATC
