File: _saved_AG_TOOL#1.sch (KiCad schematic (older format))
At the start: 35 parts, among them J1 CONN_01X03, P1 CONN_01X03, P2 CONN_01X02, Q1 Q_NPN_Darlington_BCE, Q2 Q_PMOS_DGS, SW1 SW_Push, SW2 SW_Push, SW3 SW_Push, SW4 SW_Push, SW5 SW_Push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

Commit message: changed some parts
Parts:
- DS1: footprint Pin_Headers:Pin_Header_Angled_2x16_Pitch2.00mm -> Pin_Headers:Pin_Header_Straight_1x16_Pitch2.00mm
Changed lines of the file:
@@
 F 0 "DS1" H 1900 4600 50  0000 C CNN
 F 1 "LCD16X2" H 3400 4600 50  0000 C CNN
-F 2 "Pin_Headers:Pin_Header_Angled_2x16_Pitch2.00mm" H 2700 4150 50  0001 C CIN
+F 2 "Pin_Headers:Pin_Header_Straight_1x16_Pitch2.00mm" H 2700 4150 50  0001 C CIN
 F 3 "" H 2700 4200 50  0000 C CNN
 	1    2700 4200
